Commit message: Added velodyne lidar to simulation, added rviz to launch file with config, and moved velodyne folder into the catkin_ws (This can eventually be gutted and put into one folder)

File: catkin_ws/src/navigation/gc_testing/gc_testing_description/urdf/custom.urdf.xacro (robot description, xacro)
@@ -1,4 +1,4 @@
 <?xml version="1.0"?>
-<robot name="tortoisebot">
+<robot xmlns:xacro="http://www.ros.org/wiki/xacro" name="tortoisebot">
   <link name="base_link">
     <visual>
@@ -121,4 +121,8 @@
     <origin rpy="-1.5708 0 0" xyz="-1.1685 0.5 -0.889"/>
   </joint>
+  <xacro:include filename="$(find velodyne_description)/urdf/VLP-16.urdf.xacro"/>
+  <VLP-16 parent="base_link" name="velodyne" topic="/velodyne_points" hz="10" samples="440">
+    <origin xyz="0 0 0.889" rpy="0 0 0" />
+  </VLP-16>
   <gazebo>
     <plugin name="differential_drive_controller"
