Commit message: Got motors endpoint working

File: catkin_ws/src/navigation/gc_testing/gc_testing_description/urdf/custom-backup.urdf.xacro (robot description, xacro)
@@ -5,5 +5,5 @@
       <geometry>
         <!-- l w h 2.337 1.27 1.778-->
-        <box size="0.6 0.3 0.3"/>
+        <box size="2.337 1.27 1.778"/>
       </geometry>
       <material name="silver">
@@ -13,5 +13,5 @@
     <collision>
       <geometry>
-        <box size="0.6 0.3 0.3"/>
+        <box size="2.337 1.27 1.778"/>
       </geometry>
     </collision>
@@ -45,5 +45,5 @@
     <parent link="base_link"/>
     <child link="front_caster"/>
-    <origin rpy="0 0 0" xyz="0.3 0 0"/>
+    <origin rpy="0 0 0" xyz="1.1 0 -0.739"/>
   </joint>
   <link name="front_wheel">
@@ -95,5 +95,5 @@
     <parent link="base_link"/>
     <child link="right_wheel"/>
-    <origin rpy="-1.5708 0 0" xyz="-0.2825 -0.125 -0.15"/>
+    <origin rpy="-1.5708 0 0" xyz="-1.1685 -0.5 -0.889"/>
   </joint>
   <link name="left_wheel">
@@ -119,9 +119,9 @@
     <parent link="base_link"/>
     <child link="left_wheel"/>
-    <origin rpy="-1.5708 0 0" xyz="-0.28825 0.125 -0.15"/>
+    <origin rpy="-1.5708 0 0" xyz="-1.1685 0.5 -0.889"/>
   </joint>
   <xacro:include filename="$(find velodyne_description)/urdf/VLP-16.urdf.xacro"/>
   <VLP-16 parent="base_link" name="velodyne" topic="/velodyne_points" hz="10" samples="440">
-    <origin xyz="0 0 0.15" rpy="0 0 0" />
+    <origin xyz="0 0 0.889" rpy="0 0 0" />
   </VLP-16>
   <gazebo>
@@ -131,5 +131,5 @@
       <rightJoint>right_wheel_joint</rightJoint>
       <robotBaseFrame>base_link</robotBaseFrame>
-      <wheelSeparation>0.25</wheelSeparation>
+      <wheelSeparation>1.0</wheelSeparation>
       <wheelDiameter>0.07</wheelDiameter>
       <publishWheelJointState>true</publishWheelJointState>

Commit message: updated urdf file

File: catkin_ws/src/navigation/gc_testing/gc_testing_description/urdf/custom-backup.urdf.xacro (robot description, xacro)
@@ -8,5 +8,5 @@
       </geometry>
       <material name="silver">
-        <color rgba="0.75 0.75 0.75 1"/>
+        <color rgba="0.75 0.75 0.75 .1"/>
       </material>
     </visual>
@@ -17,9 +17,17 @@
     </collision>
     <inertial>
+      <origin xyz="0 0 -1.6" rpy="0 0 0"/>
       <mass value="1.0"/>
-      <inertia ixx="0.015" iyy="0.0375" izz="0.0375"
+      <inertia ixx="0.136" iyy="0.456" izz="0.587"
                ixy="0" ixz="0" iyz="0"/>
     </inertial>
   </link>
+  <joint name="front_caster_joint" type="continuous">
+  <!--  <limit effort="30" velocity="0.5" lower="-0.785398" upper="0.785398" />-->
+    <axis xyz="0 0 1"/>
+    <parent link="base_link"/>
+    <child link="front_caster"/>
+    <origin rpy="0 0 0" xyz="1.1 0 -0.739"/>
+  </joint>
   <link name="front_caster">
     <visual>
@@ -40,15 +48,32 @@
     </inertial>
   </link>
-  <joint name="front_caster_joint" type="revolute">
-    <limit effort="30" velocity="0.5" lower="-0.785398" upper="0.785398" />
+  <joint name="caster_to_caster_rod" type="fixed">
+    <parent link="front_caster"/>
+    <child link="front_caster_rod"/>
+    <origin xyz="-.3 0 0"/>
+  </joint>
+  <link name="front_caster_rod">
+    <visual>
+      <geometry>
+        <box size="0.3 0.1 0.1"/>
+      </geometry>
+      <material name="silver"/>
+    </visual>
+    <inertial>
+      <mass value="0.1"/>
+      <inertia ixx="0.000167" iyy="0.00083" izz="0.00083"
+               ixy="0" ixz="0" iyz="0"/>
+    </inertial>
+  </link>
+  <joint name="front_wheel_joint" type="continuous">
     <axis xyz="0 0 1"/>
-    <parent link="base_link"/>
-    <child link="front_caster"/>
-    <origin rpy="0 0 0" xyz="1.1 0 -0.739"/>
+    <parent link="front_caster_rod"/>
+    <child link="front_wheel"/>
+    <origin rpy="-1.5708 0 0" xyz="0.05 0 -.15"/>
   </joint>
   <link name="front_wheel">
     <visual>
       <geometry>
-        <cylinder length="0.05" radius="0.035"/>
+        <cylinder length=".05" radius="0.14"/>
       </geometry>
       <material name="black"/>
@@ -56,6 +81,14 @@
     <collision>
       <geometry>
-        <cylinder length="0.05" radius="0.035"/>
+        <cylinder length=".05" radius="0.14"/>
       </geometry>
+      <surface>
+        <friction>
+          <ode>
+            <mu>0.1</mu>
+            <mu2>0.1</mu2>
+          </ode>
+        </friction>
+      </surface>
     </collision>
     <inertial>
@@ -65,14 +98,8 @@
     </inertial>
   </link>
-  <joint name="front_wheel_joint" type="continuous">
-    <axis xyz="0 0 1"/>
-    <parent link="front_caster"/>
-    <child link="front_wheel"/>
-    <origin rpy="-1.5708 0 0" xyz="0.05 0 -.15"/>
-  </joint>
   <link name="right_wheel">
     <visual>
       <geometry>
-        <cylinder length="0.05" radius="0.035"/>
+        <cylinder length="0.15" radius="0.14"/>
       </geometry>
       <material name="black">
@@ -82,6 +109,12 @@
     <collision>
       <geometry>
-        <cylinder length="0.05" radius="0.035"/>
+        <cylinder length="0.15" radius="0.14"/>
       </geometry>
+        <friction>
+          <ode>
+            <mu>1.00</mu>
+            <mu2>1.00</mu2>
+          </ode>
+        </friction>
     </collision>
     <inertial>
@@ -100,5 +133,5 @@
     <visual>
       <geometry>
-        <cylinder length="0.05" radius="0.035"/>
+        <cylinder length="0.15" radius="0.14"/>
       </geometry>
       <material name="black"/>
@@ -106,6 +139,12 @@
     <collision>
       <geometry>
-        <cylinder length="0.05" radius="0.035"/>
+        <cylinder length="0.15" radius="0.14"/>
       </geometry>
+        <friction>
+          <ode>
+            <mu>1.00</mu>
+            <mu2>1.00</mu2>
+          </ode>
+        </friction>
     </collision>
     <inertial>
@@ -132,6 +171,8 @@
       <robotBaseFrame>base_link</robotBaseFrame>
       <wheelSeparation>1.0</wheelSeparation>
-      <wheelDiameter>0.07</wheelDiameter>
-      <publishWheelJointState>true</publishWheelJointState>
+      <wheelDiameter>0.28</wheelDiameter>
+       <wheelTorque>1.0</wheelTorque>
+       <publishWheelJointState>true</publishWheelJointState>
+       <legacyMode>false</legacyMode>
     </plugin>
   </gazebo>
