Commit message: Working on simulator updates

File: cart_simulator/testing_description/urdf/4_point_model.urdf.xacro (robot description, xacro)
@@ -23,5 +23,5 @@
       <geometry>
         <!-- <box size="2.337 1.27 1.778"/> -->
-        <mesh filename="file:///home/nathan_moore/.gazebo/models/golf_cart/meshes/golf_cart_blender.dae" scale="1.25 1.25 1.25"/>
+        <mesh filename="file:///home/banghajs/.gazebo/models/golf_cart/meshes/golf_cart_blender.dae" scale="1.25 1.25 1.25"/>
       </geometry>
       <material name="silver">

Commit message: Removed navigation and changed 4_point_model

File: cart_simulator/testing_description/urdf/4_point_model.urdf.xacro (robot description, xacro)
@@ -23,5 +23,5 @@
       <geometry>
         <!-- <box size="2.337 1.27 1.778"/> -->
-        <mesh filename="file:///home/banghajs/.gazebo/models/golf_cart/meshes/golf_cart_blender.dae" scale="1.25 1.25 1.25"/>
+        <mesh filename="file:///home/jeffercize/.gazebo/models/golf_cart/meshes/golf_cart_blender.dae" scale="1.25 1.25 1.25"/>
       </geometry>
       <material name="silver">

Commit message: Split launch file working environments to better accomodate different settings. Fixed velodyne and base_link transform issues.

File: cart_simulator/testing_description/urdf/4_point_model.urdf.xacro (robot description, xacro)
@@ -23,5 +23,5 @@
       <geometry>
         <!-- <box size="2.337 1.27 1.778"/> -->
-        <mesh filename="file:///home/jeffercize/.gazebo/models/golf_cart/meshes/golf_cart_blender.dae" scale="1.25 1.25 1.25"/>
+        <mesh filename="file:///home/tyree/.gazebo/models/golf_cart/meshes/golf_cart_blender.dae" scale="1.25 1.25 1.25"/>
       </geometry>
       <material name="silver">

Commit message: Added landmark name to waypoint node for integration

File: cart_simulator/testing_description/urdf/4_point_model.urdf.xacro (robot description, xacro)
@@ -23,5 +23,5 @@
       <geometry>
         <!-- <box size="2.337 1.27 1.778"/> -->
-        <mesh filename="file:///home/tyree/.gazebo/models/golf_cart/meshes/golf_cart_blender.dae" scale="1.25 1.25 1.25"/>
+        <mesh filename="file:///home/jeffercize/catkin_ws/src/ai-navigation/golf_cart/meshes/golf_cart_blender.dae" scale="1.25 1.25 1.25"/>
       </geometry>
       <material name="silver">

Commit message: readying for branch

File: cart_simulator/testing_description/urdf/4_point_model.urdf.xacro (robot description, xacro)
@@ -23,5 +23,5 @@
       <geometry>
         <!-- <box size="2.337 1.27 1.778"/> -->
-        <mesh filename="file:///home/jeffercize/catkin_ws/src/ai-navigation/golf_cart/meshes/golf_cart_blender.dae" scale="1.25 1.25 1.25"/>
+        <mesh filename="file:///home/tyree/catkin_ws/src/ai-navigation/golf_cart/meshes/golf_cart_blender.dae" scale="1.25 1.25 1.25"/>
       </geometry>
       <material name="silver">

Commit message: Motor Endpoint update

File: cart_simulator/testing_description/urdf/4_point_model.urdf.xacro (robot description, xacro)
@@ -23,5 +23,5 @@
       <geometry>
         <!-- <box size="2.337 1.27 1.778"/> -->
-        <mesh filename="file:///home/tyree/catkin_ws/src/ai-navigation/golf_cart/meshes/golf_cart_blender.dae" scale="1.25 1.25 1.25"/>
+        <mesh filename="file:///home/jeffercize/catkin_ws/src/ai-navigation/golf_cart/meshes/golf_cart_blender.dae" scale="1.25 1.25 1.25"/>
       </geometry>
       <material name="silver">

Commit message: Added bus_route_design.py navigation planning

File: cart_simulator/testing_description/urdf/4_point_model.urdf.xacro (robot description, xacro)
@@ -23,5 +23,5 @@
       <geometry>
         <!-- <box size="2.337 1.27 1.778"/> -->
-        <mesh filename="file:///home/tyree/catkin_ws/src/ai-navigation/golf_cart/meshes/golf_cart_blender.dae" scale="1.25 1.25 1.25"/>
+        <mesh filename="file:///home/channathan/catkin_ws/src/ai-navigation/golf_cart/meshes/golf_cart_blender.dae" scale="1.25 1.25 1.25"/>
       </geometry>
       <material name="silver">

Commit message: Wenesday Before Dry RUn

File: cart_simulator/testing_description/urdf/4_point_model.urdf.xacro (robot description, xacro)
@@ -23,5 +23,5 @@
       <geometry>
         <!-- <box size="2.337 1.27 1.778"/> -->
-        <mesh filename="file:///home/channathan/catkin_ws/src/ai-navigation/golf_cart/meshes/golf_cart_blender.dae" scale="1.25 1.25 1.25"/>
+        <mesh filename="file:///home/jeffercize/catkin_ws/src/ai-navigation/golf_cart/meshes/golf_cart_blender.dae" scale="1.25 1.25 1.25"/>
       </geometry>
       <material name="silver">

Commit message: Motor Endpoint using Electronic/Sensor teleop.py

File: cart_simulator/testing_description/urdf/4_point_model.urdf.xacro (robot description, xacro)
@@ -23,5 +23,5 @@
       <geometry>
         <!-- <box size="2.337 1.27 1.778"/> -->
-        <mesh filename="file:///home/jeffercize/catkin_ws/src/ai-navigation/golf_cart/meshes/golf_cart_blender.dae" scale="1.25 1.25 1.25"/>
+        <mesh filename="file:///home/channathan/catkin_ws/src/ai-navigation/golf_cart/meshes/golf_cart_blender.dae" scale="1.25 1.25 1.25"/>
       </geometry>
       <material name="silver">

Commit message: Enabled obstacle detection, roughly working, ros_client needs a state fix when arriving to pick up passenger the second time. All else should be good

File: cart_simulator/testing_description/urdf/4_point_model.urdf.xacro (robot description, xacro)
@@ -23,5 +23,5 @@
       <geometry>
         <!-- <box size="2.337 1.27 1.778"/> -->
-        <mesh filename="file:///home/channathan/catkin_ws/src/ai-navigation/golf_cart/meshes/golf_cart_blender.dae" scale="1.25 1.25 1.25"/>
+        <mesh filename="file:///home/jeffercize/catkin_ws/src/ai-navigation/golf_cart/meshes/golf_cart_blender.dae" scale="1.25 1.25 1.25"/>
       </geometry>
       <material name="silver">
@@ -271,4 +271,28 @@
     <origin rpy="-1.5708 0 0" xyz="-1.1685 0.5 -0.889"/>
   </joint>
+  <!--Begin RPLidar URDF Config-->
+  <joint name="laser" type="fixed">
+    <origin xyz="1.2 0 -0.5" rpy = "0 0 3.14159"/>
+    <parent link="base_link"/>
+    <child link="base_laser_link"/>
+  </joint>
+  <link name="base_laser_link">
+    <visual>
+      <geometry>
+        <cylinder length="0.05" radius="0.05"/>
+      </geometry>
+      <material name="blue">
+        <color rgba="0 0 0.8 1"/>
+      </material>
+    </visual>
+    <intertial>
+      <mass value="0.000001"/>
+      <origin xyz="0 0 0"/>
+      <inertia ixx="0.0001" ixy="0.0" ixz="0.0"
+      iyy="0.0001" iyz="0.0"
+      izz="0.0001"/>
+    </intertial>
+  </link>
+  <!--End RPLidar stuff - Credit: Elaine Wu of SeeedBlog-->
   <!-- Velodyne lidar plugin, located on the golf cart roof -->
   <xacro:include filename="$(find velodyne_description)/urdf/VLP-16.urdf.xacro"/>

Commit message: Launch file simplifications. Path creation tool expanding functionality through new rad types. Begin moving file locations and parameters to parameter server.

File: cart_simulator/testing_description/urdf/4_point_model.urdf.xacro (robot description, xacro)
@@ -23,5 +23,5 @@
       <geometry>
         <!-- <box size="2.337 1.27 1.778"/> -->
-        <mesh filename="file:///home/jeffercize/catkin_ws/src/ai-navigation/golf_cart/meshes/golf_cart_blender.dae" scale="1.25 1.25 1.25"/>
+        <mesh filename="file:///home/browermb/catkin_ws/src/ai-navigation/golf_cart/meshes/golf_cart_blender.dae" scale="1.25 1.25 1.25"/>
       </geometry>
       <material name="silver">

Commit message: bug fixes

File: cart_simulator/testing_description/urdf/4_point_model.urdf.xacro (robot description, xacro)
@@ -23,5 +23,5 @@
       <geometry>
         <!-- <box size="2.337 1.27 1.778"/> -->
-        <mesh filename="file:///home/browermb/catkin_ws/src/ai-navigation/golf_cart/meshes/golf_cart_blender.dae" scale="1.25 1.25 1.25"/>
+        <mesh filename="file:///home/jeffercize/catkin_ws/src/ai-navigation/golf_cart/meshes/golf_cart_blender.dae" scale="1.25 1.25 1.25"/>
       </geometry>
       <material name="silver">

Commit message: Big laptop system

File: cart_simulator/testing_description/urdf/4_point_model.urdf.xacro (robot description, xacro)
@@ -23,5 +23,5 @@
       <geometry>
         <!-- <box size="2.337 1.27 1.778"/> -->
-        <mesh filename="file:///home/jeffercize/catkin_ws/src/ai-navigation/golf_cart/meshes/golf_cart_blender.dae" scale="1.25 1.25 1.25"/>
+        <mesh filename="file:///home/jacart/catkin_ws/src/ai-navigation/golf_cart/meshes/golf_cart_blender.dae" scale="1.25 1.25 1.25"/>
       </geometry>
       <material name="silver">
